File: miniRGBii.kicad_sch (KiCad schematic)
At the start: 31 parts, among them J1 Conn_01x01_Male, J2 Conn_01x01_Male, J3 Conn_01x01_Male, J4 Conn_01x01_Male, J5 Conn_01x01_Male, J6 Conn_01x01_Male, J7 Conn_01x01_Male, J8 Conn_01x01_Male, J9 Conn_01x01_Male

Commit message: Include Bill Of Materials
Signed-off-by: Devnol <pgkoutsoumanis@gmail.com>
Parts:
- removed C62, C79, C86: 50pF, symbol Device:C
Other:
- note added: "RVL-CPU-30 and earlier boards utilises 50pF unpolarized capacitors numbered C62, C79 and C86 instead of D1-D3. Knowing the value of either is trivial for completing a safe replacemement of the component video circuitry."
- note removed: "RVL-CPU-30 and earlier boards utilises capacitors instead of D1-D3. Knowing the value of either is trivial for completing a safe replacemement of the component video circuitry."
Changed lines of the file:
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@@
     (stroke (width 0) (type default) (color 0 0 0 0))
   )
-  (polyline (pts (xy 24.13 163.83) (xy 24.13 189.23))
+  (polyline (pts (xy 24.13 171.45) (xy 24.13 189.23))
     (stroke (width 0) (type default) (color 0 0 0 0))
   )
@@
     (stroke (width 0) (type default) (color 0 0 0 0))
   )
-  (polyline (pts (xy 85.09 163.83) (xy 24.13 163.83))
+  (polyline (pts (xy 85.09 171.45) (xy 24.13 171.45))
     (stroke (width 0) (type default) (color 0 0 0 0))
   )
@@
     (stroke (width 0) (type default) (color 0 0 0 0))
   )
-  (polyline (pts (xy 85.09 189.23) (xy 85.09 163.83))
+  (polyline (pts (xy 85.09 189.23) (xy 85.09 171.45))
     (stroke (width 0) (type default) (color 0 0 0 0))
   )
@@
     (stroke (width 0) (type default) (color 0 0 0 0))
   )
-  (text "RVL-CPU-30 and earlier boards utilises capacitors\ninstead of D1-D3. \nKnowing the value of either is trivial\nfor completing a safe replacemement\nof the component video circuitry."
+  (text "RVL-CPU-30 and earlier boards utilises\n50pF unpolarized capacitors\nnumbered C62, C79 and C86 instead of D1-D3. \nKnowing the value of either is trivial\nfor completing a safe replacemement\nof the component video circuitry."
     (at 25.4 185.42 0)
     (effects (font (size 1.27 1.27)) (justify left bottom))
@@
     )
   )
-  (symbol (lib_id "Device:C") (at 33.02 170.18 270) (unit 1)
-    (in_bom yes) (on_board yes)
-    (property "Reference" "C86" (id 0) (at 34.1884 173.101 90)
-      (effects (font (size 1.27 1.27)) (justify left))
-    )
-    (property "Value" "50pF" (id 1) (at 31.877 173.101 0)
-      (effects (font (size 1.27 1.27)) (justify left) hide)
-    )
-    (property "Footprint" "" (id 2) (at 29.21 171.1452 0)
-      (effects (font (size 1.27 1.27)) hide)
-    )
-    (property "Datasheet" "~" (id 3) (at 33.02 170.18 0)
-      (effects (font (size 1.27 1.27)) hide)
-    )
-    (pin "1")
-    (pin "2")
-  )
-  (symbol (lib_id "Device:C") (at 54.61 170.18 270) (unit 1)
-    (in_bom yes) (on_board yes)
-    (property "Reference" "C79" (id 0) (at 55.7784 173.101 90)
-      (effects (font (size 1.27 1.27)) (justify left))
-    )
-    (property "Value" "50pF" (id 1) (at 53.467 173.101 0)
-      (effects (font (size 1.27 1.27)) (justify left) hide)
-    )
-    (property "Footprint" "" (id 2) (at 50.8 171.1452 0)
-      (effects (font (size 1.27 1.27)) hide)
-    )
-    (property "Datasheet" "~" (id 3) (at 54.61 170.18 0)
-      (effects (font (size 1.27 1.27)) hide)
-    )
-    (pin "1")
-    (pin "2")
-  )
   (symbol (lib_id "Device:C") (at 163.83 109.22 90) (mirror x) (unit 1)
     (in_bom yes) (on_board yes)
@@
     )
     (property "Datasheet" "~" (id 3) (at 163.83 109.22 0)
-      (effects (font (size 1.27 1.27)) hide)
-    )
-    (pin "1")
-    (pin "2")
-  )
-  (symbol (lib_id "Device:C") (at 76.2 170.18 270) (unit 1)
-    (in_bom yes) (on_board yes)
-    (property "Reference" "C62" (id 0) (at 77.3684 173.101 90)
-      (effects (font (size 1.27 1.27)) (justify left))
-    )
-    (property "Value" "50pF" (id 1) (at 75.057 173.101 0)
-      (effects (font (size 1.27 1.27)) (justify left) hide)
-    )
-    (property "Footprint" "" (id 2) (at 72.39 171.1452 0)
-      (effects (font (size 1.27 1.27)) hide)
-    )
-    (property "Datasheet" "~" (id 3) (at 76.2 170.18 0)
       (effects (font (size 1.27 1.27)) hide)
     )
@@
       (reference "#PWR0111") (unit 1) (value "GND") (footprint "")
     )
-    (path "/00000000-0000-0000-0000-00005ecd629c"
-      (reference "C62") (unit 1) (value "50pF") (footprint "")
-    )
     (path "/00000000-0000-0000-0000-00005ed1e557"
       (reference "C64") (unit 1) (value "220μF") (footprint "Capacitor_Tantalum_SMD:CP_EIA-7343-15_Kemet-W_Pad2.25x2.55mm_HandSolder")
@@
       (reference "C78") (unit 1) (value "100pF") (footprint "Capacitor_SMD:C_0603_1608Metric_Pad1.05x0.95mm_HandSolder")
     )
-    (path "/00000000-0000-0000-0000-00005ecd5e01"
-      (reference "C79") (unit 1) (value "50pF") (footprint "")
-    )
     (path "/00000000-0000-0000-0000-00005ecf6bb9"
       (reference "C83") (unit 1) (value "50pF") (footprint "Capacitor_SMD:C_0603_1608Metric_Pad1.05x0.95mm_HandSolder")
@@
       (reference "C85") (unit 1) (value "100pF") (footprint "Capacitor_SMD:C_0603_1608Metric_Pad1.05x0.95mm_HandSolder")
     )
-    (path "/00000000-0000-0000-0000-00005ecd5101"
-      (reference "C86") (unit 1) (value "50pF") (footprint "")
-    )
     (path "/00000000-0000-0000-0000-00005f035767"

Commit message: Change cap footprint to reduce board size
Signed-off-by: Devnol <pgkoutsoumanis@gmail.com>
Parts:
- C64, C69, C84: footprint Capacitor_Tantalum_SMD:CP_EIA-7343-15_Kemet-W_Pad2.25x2.55mm_HandSolder -> Capacitor_Tantalum_SMD:CP_EIA-3528-12_Kemet-T_Pad1.50x2.35mm_HandSolder
Changed lines of the file:
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@@
       (effects (font (size 1.27 1.27)) (justify right))
     )
-    (property "Footprint" "Capacitor_Tantalum_SMD:CP_EIA-7343-15_Kemet-W_Pad2.25x2.55mm_HandSolder" (id 2) (at 144.78 101.2952 0)
+    (property "Footprint" "Capacitor_Tantalum_SMD:CP_EIA-3528-12_Kemet-T_Pad1.50x2.35mm_HandSolder" (id 2) (at 144.78 101.2952 0)
       (effects (font (size 1.27 1.27)) hide)
     )
@@
       (effects (font (size 1.27 1.27)) (justify right))
     )
-    (property "Footprint" "Capacitor_Tantalum_SMD:CP_EIA-7343-15_Kemet-W_Pad2.25x2.55mm_HandSolder" (id 2) (at 144.78 70.8152 0)
+    (property "Footprint" "Capacitor_Tantalum_SMD:CP_EIA-3528-12_Kemet-T_Pad1.50x2.35mm_HandSolder" (id 2) (at 144.78 70.8152 0)
       (effects (font (size 1.27 1.27)) hide)
     )
@@
       (effects (font (size 1.27 1.27)) (justify right))
     )
-    (property "Footprint" "Capacitor_Tantalum_SMD:CP_EIA-7343-15_Kemet-W_Pad2.25x2.55mm_HandSolder" (id 2) (at 144.78 39.0652 0)
+    (property "Footprint" "Capacitor_Tantalum_SMD:CP_EIA-3528-12_Kemet-T_Pad1.50x2.35mm_HandSolder" (id 2) (at 144.78 39.0652 0)
       (effects (font (size 1.27 1.27)) hide)
     )
@@
     )
     (path "/00000000-0000-0000-0000-00005ed1e557"
-      (reference "C64") (unit 1) (value "220μF") (footprint "Capacitor_Tantalum_SMD:CP_EIA-7343-15_Kemet-W_Pad2.25x2.55mm_HandSolder")
+      (reference "C64") (unit 1) (value "220μF") (footprint "Capacitor_Tantalum_SMD:CP_EIA-3528-12_Kemet-T_Pad1.50x2.35mm_HandSolder")
     )
     (path "/00000000-0000-0000-0000-00005ecd6281"
@@
     )
     (path "/00000000-0000-0000-0000-00005ed1dc64"
-      (reference "C69") (unit 1) (value "220μF") (footprint "Capacitor_Tantalum_SMD:CP_EIA-7343-15_Kemet-W_Pad2.25x2.55mm_HandSolder")
+      (reference "C69") (unit 1) (value "220μF") (footprint "Capacitor_Tantalum_SMD:CP_EIA-3528-12_Kemet-T_Pad1.50x2.35mm_HandSolder")
     )
     (path "/00000000-0000-0000-0000-00005ecdafcc"
@@
     )
     (path "/00000000-0000-0000-0000-00005ed1f3c6"
-      (reference "C84") (unit 1) (value "220μF") (footprint "Capacitor_Tantalum_SMD:CP_EIA-7343-15_Kemet-W_Pad2.25x2.55mm_HandSolder")
+      (reference "C84") (unit 1) (value "220μF") (footprint "Capacitor_Tantalum_SMD:CP_EIA-3528-12_Kemet-T_Pad1.50x2.35mm_HandSolder")
     )
     (path "/00000000-0000-0000-0000-00005ecf6bc3"

Commit message: Generate output files and add fab documentation
Signed-off-by: Devnol <pgkoutsoumanis@gmail.com>
Parts:
- C64, C69, C84: LCSC (none) -> C79111
- C66, C74, C83: value 50pF -> 47pF; LCSC (none) -> C1671
- C72, C78, C85: LCSC (none) -> C14858
- D1, D2, D3: LCSC (none) -> C406223
- FIL15, FIL16, FIL17: LCSC (none) -> C98095
- J1, J2, J3, J4, J5, J6, J7, J8, J9: now left out of the parts list
- R37, R39, R40: LCSC (none) -> C4275
Changed lines of the file:
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@@
       (effects (font (size 1.27 1.27)) (justify left))
     )
-    (property "Value" "50pF" (id 1) (at 166.37 115.57 90)
+    (property "Value" "47pF" (id 1) (at 166.37 115.57 90)
       (effects (font (size 1.27 1.27)) (justify left))
     )
@@
     )
     (property "Datasheet" "~" (id 3) (at 163.83 109.22 0)
+      (effects (font (size 1.27 1.27)) hide)
+    )
+    (property "LCSC" "C1671" (id 4) (at 163.83 109.22 90)
       (effects (font (size 1.27 1.27)) hide)
     )
@@
       (effects (font (size 1.27 1.27)) hide)
     )
+    (property "LCSC" "C14858" (id 4) (at 151.13 107.95 0)
+      (effects (font (size 1.27 1.27)) hide)
+    )
     (pin "1")
     (pin "2")
@@
       (effects (font (size 1.27 1.27)) (justify left))
     )
-    (property "Value" "50pF" (id 1) (at 166.37 83.82 90)
+    (property "Value" "47pF" (id 1) (at 166.37 83.82 90)
       (effects (font (size 1.27 1.27)) (justify left))
     )
@@
     )
     (property "Datasheet" "~" (id 3) (at 163.83 77.47 0)
+      (effects (font (size 1.27 1.27)) hide)
+    )
+    (property "LCSC" "C1671" (id 4) (at 163.83 77.47 90)
       (effects (font (size 1.27 1.27)) hide)
     )
@@
       (effects (font (size 1.27 1.27)) hide)
     )
+    (property "LCSC" "C14858" (id 4) (at 151.13 77.47 0)
+      (effects (font (size 1.27 1.27)) hide)
+    )
     (pin "1")
     (pin "2")
@@
       (effects (font (size 1.27 1.27)) (justify left))
     )
-    (property "Value" "50pF" (id 1) (at 166.37 52.07 90)
+    (property "Value" "47pF" (id 1) (at 166.37 52.07 90)
       (effects (font (size 1.27 1.27)) (justify left))
     )
@@
     )
     (property "Datasheet" "~" (id 3) (at 163.83 45.72 0)
+      (effects (font (size 1.27 1.27)) hide)
+    )
+    (property "LCSC" "C1671" (id 4) (at 163.83 45.72 90)
       (effects (font (size 1.27 1.27)) hide)
     )
@@
       (effects (font (size 1.27 1.27)) hide)
     )
+    (property "LCSC" "C14858" (id 4) (at 151.13 45.72 0)
+      (effects (font (size 1.27 1.27)) hide)
+    )
     (pin "1")
     (pin "2")
@@
       (effects (font (size 1.27 1.27)) (justify right) hide)
     )
+    (property "LCSC" "C79111" (id 5) (at 140.97 100.33 90)
+      (effects (font (size 1.27 1.27)) hide)
+    )
     (pin "1")
     (pin "2")
@@
       (effects (font (size 1.27 1.27)) (justify right) hide)
     )
+    (property "LCSC" "C79111" (id 5) (at 140.97 69.85 90)
+      (effects (font (size 1.27 1.27)) hide)
+    )
     (pin "1")
     (pin "2")
@@
     (property "max. Voltage" "6V" (id 4) (at 138.43 31.75 0)
       (effects (font (size 1.27 1.27)) (justify right) hide)
+    )
+    (property "LCSC" "C79111" (id 5) (at 140.97 38.1 90)
+      (effects (font (size 1.27 1.27)) hide)
     )
     (pin "1")
@@
       (effects (font (size 1.27 1.27)) hide)
     )
+    (property "LCSC" "C4275" (id 4) (at 132.08 45.72 0)
+      (effects (font (size 1.27 1.27)) hide)
+    )
     (pin "1")
     (pin "2")
@@
       (effects (font (size 1.27 1.27)) hide)
     )
+    (property "LCSC" "C4275" (id 4) (at 132.08 77.47 0)
+      (effects (font (size 1.27 1.27)) hide)
+    )
     (pin "1")
     (pin "2")
@@
       (effects (font (size 1.27 1.27)) hide)
     )
+    (property "LCSC" "C4275" (id 4) (at 132.08 107.95 0)
+      (effects (font (size 1.27 1.27)) hide)
+    )
     (pin "1")
     (pin "2")
@@
       (effects (font (size 1.27 1.27)) hide)
     )
+    (property "LCSC" "C98095" (id 4) (at 163.83 38.1 90)
+      (effects (font (size 1.27 1.27)) hide)
+    )
     (pin "1")
     (pin "2")
@@
       (effects (font (size 1.27 1.27)) hide)
     )
+    (property "LCSC" "C98095" (id 4) (at 163.83 69.85 90)
+      (effects (font (size 1.27 1.27)) hide)
+    )
     (pin "1")
     (pin "2")
@@
       (effects (font (size 1.27 1.27)) hide)
     )
+    (property "LCSC" "C98095" (id 4) (at 163.83 100.33 90)
+      (effects (font (size 1.27 1.27)) hide)
+    )
     (pin "1")
     (pin "2")
@@
       (effects (font (size 1.27 1.27)) hide)
     )
+    (property "LCSC" "C406223" (id 4) (at 176.53 46.99 0)
+      (effects (font (size 1.27 1.27)) hide)
+    )
     (pin "1")
     (pin "2")
@@
       (effects (font (size 1.27 1.27)) hide)
     )
+    (property "LCSC" "C406223" (id 4) (at 176.53 78.74 0)
+      (effects (font (size 1.27 1.27)) hide)
+    )
     (pin "1")
     (pin "2")
@@
     )
     (property "Datasheet" "" (id 3) (at 176.53 109.22 0)
+      (effects (font (size 1.27 1.27)) hide)
+    )
+    (property "LCSC" "C406223" (id 4) (at 176.53 109.22 0)
       (effects (font (size 1.27 1.27)) hide)
     )
@@
   )
   (symbol (lib_id "Connector:Conn_01x01_Male") (at 26.67 29.21 0) (unit 1)
-    (in_bom yes) (on_board yes)
+    (in_bom no) (on_board yes)
     (property "Reference" "J5" (id 0) (at 29.3624 27.0002 0)
       (effects (font (size 1.27 1.27)) hide)
@@
   )
   (symbol (lib_id "Connector:Conn_01x01_Male") (at 26.67 34.29 0) (unit 1)
-    (in_bom yes) (on_board yes)
+    (in_bom no) (on_board yes)
     (property "Reference" "J6" (id 0) (at 29.3624 32.0802 0)
       (effects (font (size 1.27 1.27)) hide)
@@
   )
   (symbol (lib_id "Connector:Conn_01x01_Male") (at 26.67 39.37 0) (unit 1)
-    (in_bom yes) (on_board yes)
+    (in_bom no) (on_board yes)
     (property "Reference" "J7" (id 0) (at 29.3624 37.1602 0)
       (effects (font (size 1.27 1.27)) hide)
@@
   )
   (symbol (lib_id "Connector:Conn_01x01_Male") (at 26.67 44.45 0) (unit 1)
-    (in_bom yes) (on_board yes)
+    (in_bom no) (on_board yes)
     (property "Reference" "J8" (id 0) (at 29.3624 42.2402 0)
       (effects (font (size 1.27 1.27)) hide)
@@
   )
   (symbol (lib_id "Connector:Conn_01x01_Male") (at 24.13 82.55 0) (unit 1)
-    (in_bom yes) (on_board yes)
+    (in_bom no) (on_board yes)
     (property "Reference" "J4" (id 0) (at 26.8224 80.3402 0)
       (effects (font (size 1.27 1.27)) hide)
@@
   )
   (symbol (lib_id "Connector:Conn_01x01_Male") (at 24.13 67.31 0) (unit 1)
-    (in_bom yes) (on_board yes)
+    (in_bom no) (on_board yes)
     (property "Reference" "J1" (id 0) (at 26.8224 65.1002 0)
       (effects (font (size 1.27 1.27)) hide)
@@
   )
   (symbol (lib_id "Connector:Conn_01x01_Male") (at 24.13 72.39 0) (unit 1)
-    (in_bom yes) (on_board yes)
+    (in_bom no) (on_board yes)
     (property "Reference" "J2" (id 0) (at 26.8224 70.1802 0)
       (effects (font (size 1.27 1.27)) hide)
@@
   )
   (symbol (lib_id "Connector:Conn_01x01_Male") (at 24.13 77.47 0) (unit 1)
-    (in_bom yes) (on_board yes)
+    (in_bom no) (on_board yes)
     (property "Reference" "J3" (id 0) (at 26.8224 75.2602 0)
       (effects (font (size 1.27 1.27)) hide)
@@
   )
   (symbol (lib_id "Connector:Conn_01x01_Male") (at 24.13 91.44 0) (unit 1)
-    (in_bom yes) (on_board yes)
+    (in_bom no) (on_board yes)
     (property "Reference" "J9" (id 0) (at 26.8224 89.2302 0)
       (effects (font (size 1.27 1.27)) hide)
@@
     )
     (path "/00000000-0000-0000-0000-00005ecd6281"
-      (reference "C66") (unit 1) (value "50pF") (footprint "Capacitor_SMD:C_0603_1608Metric_Pad1.05x0.95mm_HandSolder")
+      (reference "C66") (unit 1) (value "47pF") (footprint "Capacitor_SMD:C_0603_1608Metric_Pad1.05x0.95mm_HandSolder")
     )
     (path "/00000000-0000-0000-0000-00005ed1dc64"
@@
     )
     (path "/00000000-0000-0000-0000-00005ece76bf"
-      (reference "C74") (unit 1) (value "50pF") (footprint "Capacitor_SMD:C_0603_1608Metric_Pad1.05x0.95mm_HandSolder")
+      (reference "C74") (unit 1) (value "47pF") (footprint "Capacitor_SMD:C_0603_1608Metric_Pad1.05x0.95mm_HandSolder")
     )
     (path "/00000000-0000-0000-0000-00005ece7b2c"
@@
     )
     (path "/00000000-0000-0000-0000-00005ecf6bb9"
-      (reference "C83") (unit 1) (value "50pF") (footprint "Capacitor_SMD:C_0603_1608Metric_Pad1.05x0.95mm_HandSolder")
+      (reference "C83") (unit 1) (value "47pF") (footprint "Capacitor_SMD:C_0603_1608Metric_Pad1.05x0.95mm_HandSolder")
     )
     (path "/00000000-0000-0000-0000-00005ed1f3c6"
